File: ThinCalculator.kicad_pcb (KiCad board)
At the start: 2 copper layers, 63.5 x 128.3 mm, 76 parts, among them J1 SWD, J2 BATT, Q1 Q_PMOS_GSD, Q2 Q_PMOS_GSD, SW1 POWER, SW10 F2, SW11 DGR, SW12 COS, SW13 Y^X, SW14 8, SW15 5, SW16 2, SW17 +/-, SW18 F3, SW19 FSE, SW2 F1, SW20 TAN, SW21 SQRT, SW22 9, SW23 6, SW24 3, SW25 ., SW26 F4, SW27 RCL, SW28 LN, SW29 %, SW3 SHIFT, SW30 EXP, SW31 *, SW32 +, SW33 DROP, SW34 F5, SW35 STO, SW36 LOG, SW37 X<=>Y, SW38 <-, SW39 /, SW4 SIN, SW40 -, SW41 ENTER, SW5 a b/c, SW6 7, SW7 4, SW8 1, SW9 0, U1 AP3012, U2 Pico, U3 OLED_128x64_SSD1309, U4 MCP73831-2-OT

Commit message: production version 1.0
Parts:
- R1: value R -> 100k
- R2: value R -> 11k6
- SW1: value POWER -> SW_SPDT
- moved R9 0.64 mm to (110.2, 74.0)
- moved U2 0.64 mm to (124.2, 60.7)
- moved R10 0.63 mm to (105.8, 74.0)
- moved R6 0.63 mm to (112.8, 74.0)
- moved R7 0.63 mm to (107.7, 74.0)
- moved R8 0.63 mm to (103.9, 74.0)
Connections:
- net ~{POWER_EN} renamed POWER_EN
Routing:
- net GND: track 41.8 -> 44.4 mm
- net Net-(J1-Pad1): track 9.04 -> 11.4 mm
- net Net-(R10-Pad2): track 150.1 -> 151.0 mm
- net COL2: track 4.49 -> 5.38 mm
- net OLED_POWER_EN: track 21.6 -> 22.4 mm
- net COL1: track 5.20 -> 6.02 mm
- net +3V3: track 23.2 -> 24.0 mm
- net Net-(J1-Pad3): track 9.49 -> 10.2 mm
- net ROW7: track 132.3 -> 132.9 mm
- net RESET: track 14.3 -> 13.7 mm
- net BAT_STAT: track 24.7 -> 24.1 mm
- net SDO: track 14.3 -> 13.7 mm
- net ROW8: track 142.4 -> 143.1 mm
- net POWER_EN: track 85.3 -> 86.0 mm
- net Net-(R9-Pad2): track 172.7 -> 173.4 mm
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