File: ThinCalculator.kicad_sch (KiCad schematic)
At the start: 76 parts, among them J1 SWD, J2 BATT, Q1 Q_PMOS_GSD, Q2 Q_PMOS_GSD, SW1 SW_SPDT, SW10 F2, SW11 DGR, SW12 COS, SW13 Y^X, SW14 8, SW15 5, SW16 2, SW17 +/-, SW18 F3, SW19 FSE, SW2 F1, SW20 TAN, SW21 SQRT, SW22 9, SW23 6, SW24 3, SW25 ., SW26 F4, SW27 RCL, SW28 LN, SW29 %, SW3 SHIFT, SW30 EXP, SW31 *, SW32 +, SW33 DROP, SW34 F5, SW35 STO, SW36 LOG, SW37 X<=>Y, SW38 <-, SW39 /, SW4 SIN, SW40 -, SW41 ENTER, SW5 a b/c, SW6 7, SW7 4, SW8 1, SW9 0, U1 AP3012, U2 Pico, U3 OLED_128x64_SSD1309, U4 MCP73831-2-OT

Commit message: production version 1.0
Parts:
- R2: value R -> 11k6
Other:
- note added: "R1/R2 = 8.6 for 12V rail R1 = 100k, R2 = 11.6k"
- note removed: "R1/R2 = 8.6 for 12V rail R1 = 100k, R2 = 11.6k (Use 12k, V = 11.7V) R1 = 82k, R2 = 9.5k (use 10k, V = 11.5V) R1 = 68k, R2 = 7.9k (use 8k2, V = 11.6) R1 = 56k, R2 = 6.5k (use 6k8, V = 11.5)"
Changed lines of the file:
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@@
     (effects (font (size 1.27 1.27)) (justify left bottom))
   )
-  (text "R1/R2 = 8.6 for 12V rail\nR1 = 100k, R2 = 11.6k (Use 12k, V = 11.7V)\nR1 = 82k, R2 = 9.5k (use 10k, V = 11.5V)\nR1 = 68k, R2 = 7.9k (use 8k2, V = 11.6)\nR1 = 56k, R2 = 6.5k (use 6k8, V = 11.5)\n"
-    (at 133.35 213.36 0)
-    (effects (font (size 1.27 1.27)) (justify left bottom))
+  (text "R1/R2 = 8.6 for 12V rail\nR1 = 100k, R2 = 11.6k" (at 46.99 76.2 0)
+    (effects (font (size 1.27 1.27) italic) (justify left bottom))
   )
   (text "KEYBOARD MATRIX\n" (at 351.79 22.86 0)
@@
       (effects (font (size 1.27 1.27)) (justify left))
     )
-    (property "Value" "R" (id 1) (at 85.598 56.3122 0)
+    (property "Value" "11k6" (id 1) (at 85.598 56.3122 0)
       (effects (font (size 1.27 1.27)) (justify left))
     )
@@
     )
     (path "/0d66865d-1447-4a38-9305-fcc5f8933afd"
-      (reference "R2") (unit 1) (value "R") (footprint "Resistor_SMD:R_0603_1608Metric_Pad0.98x0.95mm_HandSolder")
+      (reference "R2") (unit 1) (value "11k6") (footprint "Resistor_SMD:R_0603_1608Metric_Pad0.98x0.95mm_HandSolder")
     )
     (path "/ac7ebae8-6efd-477d-b851-b9d006a5f04b"
