File: FrontPanel/FrontPanel/FrontPanel.kicad_pcb (KiCad board)
At the start: 2 copper layers, 65.4 x 130.2 mm, 0 parts

Commit message: production version 1.0
Other:
- outline, holes or cut-outs redrawn
